Commit message: Add nvblox and Isaac Sim example code
- Add example code using Isaac Sim environment
- Integrate nvblox for 3D mapping
- Demonstrate basic pick-and-place workflow with MoveIt

File: dsr_cumotion/srdf/m1013.srdf.xacro (robot description, xacro)
@@ -2,12 +2,12 @@
 <robot xmlns:xacro="http://www.ros.org/wiki/xacro" name="m1013">
   <xacro:arg name="model"   default="m1013"/>
-  <xacro:arg name="gripper" default="none"/>
   <xacro:property name="gripper" value="$(arg gripper)"/>
-  <xacro:if value="${gripper == 'none'}">
+  <xacro:property name="isaac_sim" value="$(arg isaac_sim)"/>
+  <xacro:if value="${gripper == 'none' and isaac_sim != 'true'}">
     <group name="manipulator">
       <chain base_link="base_link" tip_link="tool0"/>
     </group>
   </xacro:if>
-  <xacro:if value="${gripper != 'none'}">
+  <xacro:if value="${gripper != 'none' or isaac_sim == 'true'}">
     <group name="manipulator">
       <chain base_link="base_link" tip_link="grasp_frame"/>
@@ -100,3 +100,16 @@
     <disable_collisions link1="grasp_frame" link2="onrobot_vgc10_base_link" reason="Adjacent"/>
   </xacro:if>
+  <xacro:if value="${isaac_sim == 'true'}">
+    <disable_collisions link1="link_6" link2="vision_bracket" reason="Never"/>
+    <disable_collisions link1="tool0" link2="vision_bracket" reason="Adjacent"/>
+    <disable_collisions link1="tool0" link2="d435i_camera" reason="Adjacent"/>
+    <disable_collisions link1="grasp_frame" link2="tool0" reason="Never"/>
+    <disable_collisions link1="grasp_frame" link2="robotiq_85_left_finger_tip_link"  reason="Never"/>
+    <disable_collisions link1="grasp_frame" link2="robotiq_85_right_finger_tip_link" reason="Never"/>
+    <disable_collisions link1="vision_bracket" link2="tool0" reason="Adjacent"/>
+    <disable_collisions link1="vision_bracket" link2="robotiq_85_base_link" reason="Never"/>
+    <disable_collisions link1="d435i_camera" link2="vision_bracket" reason="Adjacent"/>
+    <disable_collisions link1="d435i_camera" link2="robotiq_85_left_finger_tip_link"  reason="Never"/>
+    <disable_collisions link1="d435i_camera" link2="robotiq_85_right_finger_tip_link" reason="Never"/>
+  </xacro:if>
 </robot>

File: dsr_cumotion/urdf/m1013.ros2_control.xacro (robot description, xacro)
@@ -58,5 +58,5 @@
         </command_interface>
         <state_interface name="position">
-          <param name="initial_value">0.0</param>
+          <param name="initial_value">1.57</param>
         </state_interface>
         <state_interface name="velocity"/>
@@ -86,5 +86,5 @@
         </command_interface>
         <state_interface name="position">
-          <param name="initial_value">0.0</param>
+          <param name="initial_value">1.57</param>
         </state_interface>
         <state_interface name="velocity"/>

File: dsr_cumotion/urdf/m1013.urdf.xacro (robot description, xacro)
@@ -13,7 +13,10 @@
   <xacro:arg name="update_rate"  default=""/>
   <xacro:property name="gripper" value="$(arg gripper)"/>
+  <xacro:arg name="isaac_sim" default="false"/>
   <!-- <xacro:property name="mode" value="$(arg mode)"/> -->
   <xacro:include filename="$(find dsr_cumotion)/urdf/macro.m1013.white.xacro"/>
-  <xacro:m1013 namespace="$(arg namespace)"/>
+  <xacro:m1013
+    namespace="$(arg namespace)"
+    isaac_sim="$(arg isaac_sim)"/>
   <xacro:if value="${gripper == 'vgc10'}">
     <xacro:include filename="$(find dsr_cumotion)/urdf/vgc10/onrobot_vgc10_4cups_model.urdf"/>

File: dsr_cumotion/urdf/macro.m1013.white.xacro (robot description, xacro)
@@ -7,9 +7,9 @@
   <xacro:property name="vision_bracket_mesh"
                 value="package://dsr_cumotion/meshes/camera_bracket/vision_bracket.dae"/>  <xacro:property name="vision_bracket_origin_xyz" value="0 0 -0.004"/>
-  <xacro:property name="vision_bracket_origin_rpy" value="0 0 0"/>
+  <xacro:property name="vision_bracket_origin_rpy" value="0 0 1.57"/>
   <xacro:property name="d435_mesh" value="package://dsr_cumotion/meshes/camera_bracket/d435.dae"/>
   <xacro:property name="d435_joint_xyz" value="0 0.12 0.0455"/>
   <xacro:property name="d435_joint_rpy" value="0 0 0"/>
-  <xacro:macro name="m1013" params="namespace">
+  <xacro:macro name="m1013" params="namespace isaac_sim">
     <xacro:dsr_materials/>
     <link name="base_link">
@@ -38,5 +38,5 @@
       <origin rpy="0 0 0" xyz="0 0 0.1525"/>
       <axis xyz="0 0 1"/>
-      <limit effort="346" lower="-6.2832" upper="6.2832" velocity="2.0944"/>
+      <limit effort="346" lower="-3.14" upper="3.14" velocity="2.0944"/>
       <dynamics friction="0"/>
     </joint>
@@ -66,5 +66,5 @@
       <origin rpy="0 -1.571 -1.571" xyz="0 0.0345 0"/>
       <axis xyz="0 0 1"/>
-      <limit effort="346" lower="-6.2832" upper="6.2832" velocity="2.0944"/>
+      <limit effort="346" lower="-1.3" upper="1.3" velocity="2.0944"/>
       <dynamics friction="0"/>
     </joint>
@@ -118,5 +118,5 @@
       <origin rpy="0 0 1.571" xyz="0.62 0 0"/>
       <axis xyz="0 0 1"/>
-      <limit effort="163" lower="-2.7925" upper="2.7925" velocity="3.1416"/>
+      <limit effort="163" lower="-2.0" upper="2.0" velocity="3.1416"/>
       <dynamics friction="0"/>
     </joint>
@@ -146,5 +146,5 @@
       <origin rpy="1.571 0 0" xyz="0 -0.559 0"/>
       <axis xyz="0 0 1"/>
-      <limit effort="50" lower="-6.2832" upper="6.2832" velocity="3.927"/>
+      <limit effort="50" lower="-3.14" upper="3.14" velocity="3.927"/>
       <dynamics friction="0"/>
     </joint>
@@ -186,5 +186,5 @@
       <origin rpy="-1.571 0 0" xyz="0 0 0"/>
       <axis xyz="0 0 1"/>
-      <limit effort="50" lower="-6.2832" upper="6.2832" velocity="3.927"/>
+      <limit effort="50" lower="-2.0" upper="2.0" velocity="3.927"/>
       <dynamics friction="0"/>
     </joint>
@@ -214,5 +214,5 @@
       <origin rpy="1.571 0 0" xyz="0 -0.121 0"/>
       <axis xyz="0 0 1"/>
-      <limit effort="50" lower="-6.2832" upper="6.2832" velocity="3.927"/>
+      <limit effort="50" lower="-3.14" upper="3.14" velocity="3.927"/>
       <dynamics friction="0"/>
     </joint>
@@ -249,30 +249,32 @@
       <child  link="gripper_frame"/>
     </joint>
-    <!-- <joint name="vision_bracket_joint" type="fixed">
-      <parent link="tool0"/>
-      <child link="vision_bracket"/>
-      <origin xyz="${vision_bracket_origin_xyz}" rpy="${vision_bracket_origin_rpy}"/>
-    </joint>
-    <link name="vision_bracket">
-      <visual>
-        <origin xyz="0 0 0" rpy="0 0 0"/>
-        <geometry>
-          <mesh filename="${vision_bracket_mesh}"/>
-        </geometry>
-      </visual>
-    </link>
-    <joint name="d435i_camera_joint" type="fixed">
-      <parent link="vision_bracket"/>
-      <child link="d435i_camera"/>
-      <origin xyz="${d435_joint_xyz}" rpy="${d435_joint_rpy}"/>
-    </joint>
-    <link name="d435i_camera">
-      <visual>
-        <origin xyz="0 0 0" rpy="0 0 0"/>
-        <geometry>
-          <mesh filename="${d435_mesh}"/>
-        </geometry>
-      </visual>
-    </link> -->
+    <xacro:if value="${isaac_sim}">
+      <joint name="vision_bracket_joint" type="fixed">
+        <parent link="tool0"/>
+        <child link="vision_bracket"/>
+        <origin xyz="${vision_bracket_origin_xyz}" rpy="${vision_bracket_origin_rpy}"/>
+      </joint>
+      <link name="vision_bracket">
+        <visual>
+          <origin xyz="0 0 0" rpy="0 0 0"/>
+          <geometry>
+            <mesh filename="${vision_bracket_mesh}"/>
+          </geometry>
+        </visual>
+      </link>
+      <joint name="d435i_camera_joint" type="fixed">
+        <parent link="vision_bracket"/>
+        <child link="d435i_camera"/>
+        <origin xyz="${d435_joint_xyz}" rpy="${d435_joint_rpy}"/>
+      </joint>
+      <link name="d435i_camera">
+        <visual>
+          <origin xyz="0 0 0" rpy="0 0 0"/>
+          <geometry>
+            <mesh filename="${d435_mesh}"/>
+          </geometry>
+        </visual>
+      </link>
+    </xacro:if>
     <xacro:dsr_transmission/>
     <xacro:dsr_gazebo namespace="${namespace}"/>

File: dsr_cumotion/urdf/robotiq/robotiq.xacro (robot description, xacro)
@@ -154,5 +154,5 @@
     <link name="grasp_frame">
       <inertial>
-        <origin xyz="0 0 0" rpy="0 0 0"/>
+        <origin xyz="0 0 0" rpy="0 0 3.14"/>
         <mass value="0.01"/>
         <inertia ixx="0.0001" ixy="0.0" ixz="0.0" iyy="0.0001" iyz="0.0" izz="0.0001"/>
